File: zenith-pcba/untitled.kicad_sch (KiCad schematic)
At the start: 1 part, among them U1 XC7A50T-CSG325

Commit message: feat(pcba): initial programmer setup
Parts:
- removed U1: XC7A50T-CSG325, Package_BGA:Xilinx_CSG325, symbol FPGA_Xilinx_Artix7:XC7A50T-CSG325
